File: STM32_Adapter.kicad_pcb (KiCad board)
At the start: 2 copper layers, 47 x 69 mm, 17 parts, among them J101 PinHeader_02X25, J102 PinHeader_02X25, U101 STM32F072V8T6, U102 SIP21106, Y101 Crystal_smd_11x5, Y102 Crystal_smd_32768_horizontal

Commit message: pcb plokstes paruosimas
Parts:
- added C1: C_100n_0805_X7R, capacitors:C_0805, F.Cu at (154.9, 90.5)
- added C109: C_100n_0805_X7R, capacitors:C_0805, F.Cu at (147.1, 89.2)
- added C110: C_100n_0805_X7R, capacitors:C_0805, F.Cu at (133.9, 135.4)
- added D1: D_BAS85, disc:D_MiniMELF, F.Cu at (154.9, 85.8)
- added D2: EL19-21SYGC, disc:LED_0603, F.Cu at (149.0, 121.7)
- added D3: EL19-21SYGC, disc:LED_0603, F.Cu at (145.5, 121.8)
- added JP1: Jumper, mech:SMD_Jumper, B.Cu at (159.6, 118.1)
- added JP101: Jumper, mech:SMD_Jumper, B.Cu at (134.1, 83.8)
- added JP102: Jumper, mech:SMD_Jumper, B.Cu at (134.1, 85.1)
- added JP103: Jumper, mech:SMD_Jumper, B.Cu at (134.1, 88.9)
- added JP104: Jumper, mech:SMD_Jumper, B.Cu at (134.1, 90.1)
- added JP2: Jumper, mech:SMD_Jumper, B.Cu at (159.6, 116.8)
- added R1: R_470_0805_1%, resistors:R_0805, F.Cu at (137.0, 76.7)
- added R2: R_10k_0805_1%, resistors:R_0805, F.Cu at (157.4, 88.2)
- added R3: R_120_0805_1%, resistors:R_0805, F.Cu at (157.4, 84.8)
- added R4: R_1k_0805_1%, resistors:R_0805, F.Cu at (149.0, 118.7)
- added R5: R_1k_0805_1%, resistors:R_0805, F.Cu at (145.5, 118.7)
- added REF**: Measurement_Point_Square-TH_Small, Measurement_Points:Measurement_Point_Square-TH_Small, F.Cu at (147.3, 120.3)
- added REF**: Measurement_Point_Square-TH_Small, Measurement_Points:Measurement_Point_Square-TH_Small, F.Cu at (161.8, 106.7)
- added REF**: Measurement_Point_Square-TH_Small, Measurement_Points:Measurement_Point_Square-TH_Small, F.Cu at (158.5, 104.1)
- added REF**: Measurement_Point_Square-TH_Small, Measurement_Points:Measurement_Point_Square-TH_Small, F.Cu at (154.3, 103.9)
- added REF**: Measurement_Point_Square-TH_Small, Measurement_Points:Measurement_Point_Square-TH_Small, F.Cu at (151.8, 107.4)
- added REF**: Measurement_Point_Square-TH_Small, Measurement_Points:Measurement_Point_Square-TH_Small, F.Cu at (148.5, 98.7)
- added REF**: Measurement_Point_Square-TH_Small, Measurement_Points:Measurement_Point_Square-TH_Small, F.Cu at (143.9, 102.7)
- added REF**: Measurement_Point_Square-TH_Small, Measurement_Points:Measurement_Point_Square-TH_Small, F.Cu at (133.6, 105.9)
- added REF**: Measurement_Point_Square-TH_Small, Measurement_Points:Measurement_Point_Square-TH_Small, F.Cu at (141.5, 107.3)
- added REF**: Measurement_Point_Square-TH_Small, Measurement_Points:Measurement_Point_Square-TH_Small, F.Cu at (144.7, 110.6)
- added REF**: Measurement_Point_Square-TH_Small, Measurement_Points:Measurement_Point_Square-TH_Small, F.Cu at (133.0, 130.3)
- added REF**: Measurement_Point_Square-TH_Small, Measurement_Points:Measurement_Point_Square-TH_Small, F.Cu at (132.2, 102.7)
- added REF**: Measurement_Point_Square-TH_Small, Measurement_Points:Measurement_Point_Square-TH_Small, F.Cu at (132.5, 133.4)
- added REF**: Measurement_Point_Square-TH_Small, Measurement_Points:Measurement_Point_Square-TH_Small, F.Cu at (162.6, 139.7)
- added REF**: Measurement_Point_Square-TH_Small, Measurement_Points:Measurement_Point_Square-TH_Small, F.Cu at (157.5, 139.7)
- added REF**: Measurement_Point_Square-TH_Small, Measurement_Points:Measurement_Point_Square-TH_Small, F.Cu at (152.4, 139.7)
- added REF**: Measurement_Point_Square-TH_Small, Measurement_Points:Measurement_Point_Square-TH_Small, F.Cu at (147.3, 139.7)
- added REF**: Measurement_Point_Square-TH_Small, Measurement_Points:Measurement_Point_Square-TH_Small, F.Cu at (142.2, 139.7)
- added REF**: Measurement_Point_Square-TH_Small, Measurement_Points:Measurement_Point_Square-TH_Small, F.Cu at (137.2, 139.7)
- added REF**: Measurement_Point_Square-TH_Small, Measurement_Points:Measurement_Point_Square-TH_Small, F.Cu at (158.3, 73.7)
- added REF**: Measurement_Point_Square-TH_Small, Measurement_Points:Measurement_Point_Square-TH_Small, F.Cu at (154.9, 73.7)
- added REF**: Measurement_Point_Square-TH_Small, Measurement_Points:Measurement_Point_Square-TH_Small, F.Cu at (149.9, 73.7)
- added REF**: Measurement_Point_Square-TH_Small, Measurement_Points:Measurement_Point_Square-TH_Small, F.Cu at (145.7, 107.6)
- added REF**: Measurement_Point_Square-TH_Small, Measurement_Points:Measurement_Point_Square-TH_Small, F.Cu at (143.8, 73.7)
- added REF**: Measurement_Point_Square-TH_Small, Measurement_Points:Measurement_Point_Square-TH_Small, F.Cu at (139.7, 73.7)
- added REF**: Measurement_Point_Square-TH_Small, Measurement_Points:Measurement_Point_Square-TH_Small, F.Cu at (143.1, 82.4)
- added REF**: Measurement_Point_Square-TH_Small, Measurement_Points:Measurement_Point_Square-TH_Small, F.Cu at (134.1, 82.4)
- added REF**: Measurement_Point_Square-TH_Small, Measurement_Points:Measurement_Point_Square-TH_Small, F.Cu at (132.2, 80.0)
- added REF**: Measurement_Point_Square-TH_Small, Measurement_Points:Measurement_Point_Square-TH_Small, F.Cu at (133.6, 75.2)
- added REF**: Measurement_Point_Square-TH_Small, Measurement_Points:Measurement_Point_Square-TH_Small, F.Cu at (148.5, 111.2)
- added REF**: Measurement_Point_Square-TH_Small, Measurement_Points:Measurement_Point_Square-TH_Small, F.Cu at (151.0, 80.1)
- added REF**: Measurement_Point_Square-TH_Small, Measurement_Points:Measurement_Point_Square-TH_Small, F.Cu at (136.9, 92.1)
- added REF**: Measurement_Point_Square-TH_Small, Measurement_Points:Measurement_Point_Square-TH_Small, F.Cu at (149.2, 82.5)
- added REF**: Measurement_Point_Square-TH_Small, Measurement_Points:Measurement_Point_Square-TH_Small, F.Cu at (160.0, 88.8)
- added REF**: Measurement_Point_Square-TH_Small, Measurement_Points:Measurement_Point_Square-TH_Small, F.Cu at (157.2, 91.1)
- moved D101 52.3 mm to (152.3, 87.7), turned to 270 degrees
- moved R101 50.6 mm to (150.1, 86.8), turned to 90 degrees
- moved C101 46.0 mm to (150.1, 90.5), turned to 270 degrees
- moved C105 18.8 mm to (136.9, 81.2), turned to 180 degrees
- moved C107 14.9 mm to (155.2, 76.7), turned to 0 degrees
- moved C108 9.77 mm to (136.9, 74.7)
- moved C102 7.66 mm to (154.9, 81.0), turned to 90 degrees
- moved C106 6.99 mm to (136.9, 83.7)
- moved C103 4.82 mm to (157.1, 81.0), turned to 90 degrees
- moved Y102 4.07 mm to (141.0, 83.7)
- moved C104 0.13 mm to (160.3, 75.6)
Connections:
- C102 pad 1: /VDD -> Net-(C102-Pad1)
- C105 pad 1: Net-(C105-Pad1) -> /OSC32IN
- C106 pad 1: Net-(C106-Pad1) -> /OSC32OUT
- C107 pad 1: Net-(C107-Pad1) -> /RCCIN
- J102 pad 10: /PB8 -> Net-(J102-Pad10)
- J102 pad 29: /PA12 -> /PA11
- J102 pad 30: /PA13 -> /PA12
- J102 pad 31: /PA10 -> /PA9
- J102 pad 32: /PA11 -> /PA10
- J102 pad 33: /PA8 -> /PC9
- J102 pad 34: /PA9 -> /PA8
- J102 pad 35: /PC8 -> /PC7
- J102 pad 36: /PC9 -> /PC8
- J102 pad 37: /PC6 -> /PD15
- J102 pad 38: /PC7 -> /PC6
- J102 pad 39: /PD14 -> /PD13
- J102 pad 40: /PD15 -> /PD14
- J102 pad 41: /PD12 -> /PD11
- J102 pad 42: /PD13 -> /PD12
- J102 pad 43: /PD10 -> /PD9
- J102 pad 44: /PD11 -> /PD10
- J102 pad 45: /PD8 -> /PB15
- J102 pad 46: /PD9 -> /PD8
- J102 pad 47: /PB14 -> /PB13
- J102 pad 48: /PB15 -> /PB14
- J102 pad 49: /PB12 -> /COM
- J102 pad 50: /PB13 -> /PB12
- J102 pad 6: Net-(J102-Pad6) -> /PE0
- J102 pad 8: /PE0 -> /PB8
- U101 pad 12: /PF0 -> /RCCIN
- U101 pad 13: /PF1 -> /RCCOUT
- U101 pad 8: /PC14 -> /OSC32IN
- U101 pad 9: /PC15 -> /OSC32OUT
- U102 pad 5: /VDD -> Net-(C102-Pad1)
- Y101 pad 1: Net-(C106-Pad1) -> Net-(C108-Pad1)
- Y101 pad 2: Net-(C105-Pad1) -> /RCCIN
- Y102 pad 1: Net-(C108-Pad1) -> /OSC32OUT
- Y102 pad 2: Net-(C107-Pad1) -> /OSC32IN
Routing:
- net /PA4: track 87.1 -> 13.5 mm
- net /~NRST: track 14.1 -> 86.2 mm, vias 1 -> 3
- net /SWDIO: track 112.0 -> 41.7 mm
- net /PA2: track 82.3 -> 12.2 mm
- net /RCCOUT: track 0.00 -> 47.4 mm, vias 0 -> 4
- net /RCCIN: track 0.00 -> 45.9 mm, vias 0 -> 4
- net /OSC32IN: track 0.00 -> 27.5 mm, vias 0 -> 2
- net /OSC32OUT: track 0.00 -> 23.4 mm, vias 0 -> 2
- net /VDD: track 64.7 -> 86.3 mm, vias 5 -> 0
- net /PC14: track 21.1 -> 4.24 mm
- net /PC15: track 23.2 -> 7.31 mm
- net Net-(JP2-Pad2): track 0.00 -> 15.7 mm, vias 0 -> 1
- net Net-(JP1-Pad2): track 0.00 -> 12.4 mm, vias 0 -> 1
- net /PF0: track 16.4 -> 4.24 mm
- net /PF1: track 19.1 -> 7.33 mm
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Other:
- board text added: "BOOT0"
- board text added: "BOOT0 COM"
- board text added: "COM"
- board text added: "PA0"
- board text added: "PA1"
- board text added: "PA10"
- board text added: "PA11"
- board text added: "PA12"
- board text added: "PA2"
- board text added: "PA3"
- board text added: "PA4"
- board text added: "PA5"
- board text added: "PA6"
- board text added: "PA7"
- board text added: "PA8"
- board text added: "PA9"
- board text added: "PB0"
- board text added: "PB1"
- board text added: "PB10"
- board text added: "PB11"
- board text added: "PB12"
- board text added: "PB13"
- board text added: "PB14"
- board text added: "PB15"
- board text added: "PB2"
- board text added: "PB3"
- board text added: "PB4"
- board text added: "PB5"
- board text added: "PB6"
- board text added: "PB7"
- board text added: "PB8"
- board text added: "PB9"
- board text added: "PC0"
- board text added: "PC1"
- board text added: "PC10"
- board text added: "PC11"
- board text added: "PC12"
- board text added: "PC13"
- board text added: "PC14"
- board text added: "PC15"
- board text added: "PC2"
- board text added: "PC3"
- board text added: "PC4"
- board text added: "PC5"
- board text added: "PC6"
- board text added: "PC7"
- board text added: "PC8"
- board text added: "PC9"
- board text added: "PD0"
- board text added: "PD1"
- board text added: "PD10"
- board text added: "PD11"
- board text added: "PD12"
- board text added: "PD13"
- board text added: "PD14"
- board text added: "PD15"
- board text added: "PD2"
- board text added: "PD3"
- board text added: "PD4"
- board text added: "PD5"
- board text added: "PD6"
- board text added: "PD7"
- board text added: "PD8"
- board text added: "PD9"
- board text added: "PE0"
- board text added: "PE1"
- board text added: "PE10"
- board text added: "PE11"
- board text added: "PE12"
- board text added: "PE13"
- board text added: "PE14"
- board text added: "PE15"
- board text added: "PE3"
- board text added: "PE5"
- board text added: "PE7"
- board text added: "PE8"
- board text added: "PE9"
- board text added: "PF0"
- board text added: "PF1"
- board text added: "PF10"
- board text added: "PF2"
- board text added: "PF3"
- board text added: "PF6"
- board text added: "PF9"
- board text added: "PWR"
- board text added: "RE2"
- board text added: "RE4"
- board text added: "RE6"
- board text added: "SWCLK"
- board text added: "SWDIO"
- board text added: "VBAT"
- board text added: "VDD"
- board text added: "VDD2"
- board text added: "VDDA"
- board text added: "~NRST"

Commit message: pcb plokstes paruosimas
Parts:
- removed the REF** at (143.9, 102.7)
- removed the REF** at (133.0, 130.3)
- removed the REF** at (145.7, 107.6)
- removed the REF** at (133.6, 75.2)
- removed the REF** at (136.9, 92.1)
- added C2: C_1u_0805_X7R, capacitors:C_1206, F.Cu at (133.8, 104.1)
- added C3: C_100n_0805_X7R, capacitors:C_0805, F.Cu at (136.1, 91.3)
- added JP3: Jumper_SMD, mech:SMD_Jumper, B.Cu at (137.9, 96.4)
- added R6: R_120_0805_1%, resistors:R_0805, F.Cu at (137.9, 93.3)
- added REF**: , Measurement_Points:Measurement_Point_Square-TH_Small, F.Cu at (131.6, 73.7)
- added REF**: Measurement_Point_Square-TH_Small, Measurement_Points:Measurement_Point_Square-TH_Small, F.Cu at (131.6, 139.7)
- added REF**: Measurement_Point_Square-TH_Small, Measurement_Points:Measurement_Point_Square-TH_Small, F.Cu at (146.9, 93.2)
- added REF**: Measurement_Point_Square-TH_Small, Measurement_Points:Measurement_Point_Square-TH_Small, F.Cu at (137.9, 90.5)
- JP1, JP101, JP102, JP103, JP104, JP2: value Jumper -> Jumper_SMD
- REF** (x7): value Measurement_Point_Square-TH_Small -> (none)
- moved REF** 12.0 mm to (141.3, 101.4)
- moved REF** 9.10 mm to (142.7, 105.0)
- moved REF** 4.53 mm to (136.5, 104.2)
- moved REF** 3.33 mm to (148.1, 85.7)
- moved REF** 1.33 mm to (150.1, 79.1)
- moved REF** 1.31 mm to (159.3, 103.1)
- moved REF** 0.85 mm to (148.7, 110.4)
- moved REF** 0.08 mm to (141.4, 107.3)
Routing:
- net /VDDA: track 13.9 -> 31.3 mm, vias 0 -> 1
- net /VDD: track 86.3 -> 100.8 mm, vias 0 -> 1
- net /~NRST: track 86.2 -> 83.8 mm, vias 3 -> 2
- net Net-(JP3-Pad2): track 0.00 -> 1.83 mm, vias 0 -> 1
- net /VBAT: track 25.7 -> 24.8 mm
- net /PE6: track 30.1 -> 29.3 mm
- net /PC10: track 11.8 -> 11.1 mm
- net /PC11: track 14.9 -> 14.2 mm
- net /RCCIN: track 45.9 -> 45.3 mm
Other:
- board text added: "PE2"
- board text added: "PE4"
- board text added: "PE6"
- board text removed: "RE2"
- board text removed: "RE4"
- board text removed: "RE6"
